File: yuv-rgb-converter.kicad_pcb (KiCad board)
At the start: 2 copper layers, 65.3 x 53.1 mm, 56 parts, among them J1 YUV IN, J2 RGB OUT, J3 POWER, Q1 BC548, Q2 BC548, Q3 BC548, Q4 BC548, Q5 BC548, Q6 BC548, Q7 BC548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

Commit message: README, original schematics
Routing:
- removed copper zone on B.Cu, net +5V
Other:
- board text added: "+5V"
- board text added: "B"
- board text added: "G"
- board text added: "GND"
- board text added: "R"
- board text added: "SYNC"
- board text added: "U"
- board text added: "V"
- board text added: "git@github.com:hanshuebner/yuv-converter"
- board text added: "~Y"

Commit message: Production files & PDF
Other:
- board text added: "Version 1"
Changed lines of the file:
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@@
   (general
     (thickness 1.6)
-    (drawings 26)
+    (drawings 27)
     (tracks 488)
     (zones 0)
@@
     )
   )
-  (gr_text git@github.com:hanshuebner/yuv-converter (at 90.424 99.568 90) (layer F.SilkS)
+  (gr_text "Version 1" (at 89.916 104.14 90) (layer F.SilkS)
+    (effects (font (size 1 1) (thickness 0.15)))
+  )
+  (gr_text git@github.com:hanshuebner/yuv-converter (at 91.694 99.568 90) (layer F.SilkS)
     (effects (font (size 1 0.5) (thickness 0.125)))
   )
